Commit message: resize food

File: data/food/food_item0.urdf (robot description, URDF)
Before this commit: robot food_item, 1 links, 0 joints
Links:
- link food_item: geometry collision box size=0.05 0.05 0.05; visual box size=0.05 0.05 0.05

File: data/food/food_item1.urdf (robot description, URDF)
Before this commit: robot food_item, 1 links, 0 joints
Links:
- link food_item: geometry collision box size=0.05 0.05 0.05; visual box size=0.05 0.05 0.05

Commit message: resize food

File: data/food/food_item0.urdf (robot description, URDF)
Before this commit: robot food_item, 1 links, 0 joints
Links:
- link food_item: geometry collision box size=0.03 0.03 0.05; visual box size=0.03 0.03 0.05

File: data/food/food_item1.urdf (robot description, URDF)
Before this commit: robot food_item, 1 links, 0 joints
Links:
- link food_item: geometry collision box size=0.03 0.03 0.05; visual box size=0.03 0.03 0.05

Commit message: adjust 3d models

File: data/food/food_item0.urdf (robot description, URDF)
Before this commit: robot food_item, 1 links, 0 joints
Links:
- removed link food_item
- added link food_item0; collision box size=0.03 0.03 0.03; visual box size=0.03 0.03 0.03

File: data/food/food_item1.urdf (robot description, URDF)
Before this commit: robot food_item, 1 links, 0 joints
Links:
- removed link food_item
- added link food_item1; collision box size=0.03 0.03 0.03; visual box size=0.03 0.03 0.03

File: data/food/food_item2.urdf (robot description, URDF)
Before this commit: robot food_item, 1 links, 0 joints
Links:
- removed link food_item
- added link food_item2; collision box size=0.05 0.05 0.05; visual box size=0.05 0.05 0.05
