Commit message: updated urdfs for kitchen envs

File: data/food/lime.urdf (robot description, URDF)
Before this commit: robot lime, 1 links, 0 joints
Links:
- link lime: geometry collision mesh filename=lime.stl scale=0.0007 0.0007 0.0007; visual mesh filename=lime.dae scale=0.0007 0.0007 0.0007

File: data/furniture/kitchen_counter.urdf (robot description, URDF)
Before this commit: robot kitchen_counter, 1 links, 0 joints
Links:
- link kitchen_counter: geometry collision box size=0.5 1.12 0.92; collision box size=0.6 1.22 0.04

File: data/furniture/sink_counter.urdf (robot description, URDF)
Before this commit: robot sink_counter, 1 links, 0 joints
Links:
- link sink_counter: geometry collision box size=0.02 0.02 0.2; collision box size=0.16 1.22 0.04

File: data/objects/bowl_green.urdf (robot description, URDF)
Before this commit: robot bowl, 1 links, 0 joints
Links:
- link bowl: geometry collision mesh filename=bowl.stl scale=1.0 1.0 1.0; visual mesh filename=bowl.stl scale=1.0 1.0 1.0

File: data/objects/cutting_board.urdf (robot description, URDF)
Before this commit: robot cutting_board, 1 links, 0 joints
Links:
- link cutting_board: geometry collision box size=.23 0.02 0.007; collision box size=.23 0.33 0.007

File: data/objects/knife_big.urdf (robot description, URDF)
Before this commit: robot knife, 1 links, 0 joints
Links:
- link knife: geometry collision mesh filename=knife.stl scale=1.6 1.6 1.6; visual mesh filename=knife.stl scale=1.6 1.6 1.6

File: data/objects/toaster.urdf (robot description, URDF)
Before this commit: robot toaster, 1 links, 0 joints
Links:
- link toaster: geometry collision mesh filename=toaster.stl scale=0.00225 0.00225 0.00225; visual mesh filename=toaster.stl scale=0.00225 0.00225 0.00225
