Commit message: added stove object

File: data/objects/cooking_pot.urdf (robot description, URDF)
Before this commit: robot cooking_pot, 1 links, 0 joints
Links:
- link body: geometry collision mesh filename=cooking_pot.stl scale=0.025 0.025 0.015; visual mesh filename=cooking_pot.stl scale=0.025 0.025 0.015

File: data/objects/skillet.urdf (robot description, URDF)
Before this commit: robot skillet, 1 links, 0 joints
Links:
- link skillet: geometry collision mesh filename=skillet.stl scale=0.2 0.2 0.2; visual mesh filename=skillet.stl scale=0.2 0.2 0.2
